File: kicad/Drossel_Pumpe/Drossel_Pumpe.sch (KiCad schematic (older format))
At the start: 7 parts, among them J1 Conn_02x01, M1 Pumpe

Commit message: geändert:       abschlussprojekt/abschlussprojekt.ino 	geändert:       kicad/Drossel_Pumpe/Drossel_Pumpe.pdf 	geändert:       kicad/Drossel_Pumpe/Drossel_Pumpe.sch 	geändert:       kicad/Drossel_Pumpe/Drossel_Pumpe.sch-bak 	geändert:       qelectrotech/verdrahtung/schematische_beschaltung.pdf 	geändert:       qelectrotech/verdrahtung/schematische_beschaltung.qet
Other:
- note added: "Leitungsfilter"
- note removed: "Filter"
Changed lines of the file:
@@
 encoding utf-8
 Sheet 1 1
-Title "Entstördrosseln für die Wasserpumpe"
-Date "2019-07-10"
+Title "Leitungsfilter für die Wasserpumpe"
+Date "2019-11-03"
 Rev "0.2"
 Comp "STB AEA8"
@@
 	5800 3350 5800 2550
 Text Notes 6250 2500 0    79   ~ 0
-Filter
+Leitungsfilter
 Text Notes 9250 1350 0    50   ~ 0
 Infos aus dem Netz:\nSpule -> 50-100µH\nKondensator -> 47-100nF
